File: PCB Stuff/midi.kicad_pcb (KiCad board)
At the start: 2 copper layers, 193 x 204 mm, 86 parts, among them SW1 SW_Push, SW10 SW_Push, SW11 SW_Push, SW12 SW_Push, SW13 SW_Push, SW14 SW_Push, SW15 SW_Push, SW16 SW_Push, SW17 SW_Push, SW18 SW_Push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

Commit message: Add files via upload
Routing:
- net GND: track 1803.2 -> 51.7 mm
- net Net-(U2-D12): track 86.5 -> 85.6 mm
- added copper zone on B.Cu, net GND
- added copper zone on F.Cu, net GND
Other:
- outline, holes or cut-outs redrawn
